File: minputer/minputer.kicad_sch (KiCad schematic)
At the start: 50 parts, among them J1 Conn_02x20_Odd_Even, J2 Conn_01x03_Male, P1 USB_C_Plug_USB2.0, SW1 SW_Push, U1 W65C22, U11 CP2102N-Axx-xQFN20, U2 16C2552_PLCC, U3 W65C816, U4 74HC02, U5 74HC00, U6 28C256, U7 74LS573, U8 DS1318, U9 AS6C4008-55PCN

Commit message: Finish schematic
Parts:
- added C10, C15, C16, C2, C3, C4, C5, C6, C7, C8, C9: 0.1u, Capacitor_THT:C_Disc_D4.3mm_W1.9mm_P5.00mm, symbol Device:C
- added C13, C14: 4.7u, Capacitor_THT:C_Disc_D4.3mm_W1.9mm_P5.00mm, symbol Device:C
- added D21, D22: LED, LED_THT:LED_D5.0mm, symbol Device:LED
- added D23, D24, D25, D26, D27, D29, D30, D31, D32, D33, D34, D35: D_TVS, symbol Device:D_TVS
- added J2: Conn_01x02_Male, symbol Connector:Conn_01x02_Male
- added J4: Conn_02x05_Odd_Even, symbol Connector_Generic:Conn_02x05_Odd_Even
- added J?: Conn_02x10_Odd_Even, symbol Connector_Generic:Conn_02x10_Odd_Even
- added R11, R12, R13, R14, R15, R16, R17, R19, R20, R23, R24, R4: 1k, Resistor_THT:R_Axial_DIN0207_L6.3mm_D2.5mm_P7.62mm_Horizontal, symbol Device:R
- added R18, R21: 330, Resistor_THT:R_Axial_DIN0207_L6.3mm_D2.5mm_P7.62mm_Horizontal, symbol Device:R
- added R22: 10k, Resistor_THT:R_Axial_DIN0207_L6.3mm_D2.5mm_P7.62mm_Horizontal, symbol Device:R
- added R26: 22.1k, Resistor_SMD:R_0603_1608Metric_Pad0.98x0.95mm_HandSolder, symbol Device:R
- added R27: 47.5k, Resistor_SMD:R_0603_1608Metric_Pad0.98x0.95mm_HandSolder, symbol Device:R
- added R28: 5.1k, Resistor_SMD:R_0603_1608Metric_Pad0.98x0.95mm_HandSolder, symbol Device:R
- added U3: 74LS138, symbol 74xx:74LS138
- C1: value C -> 0.1u
- C11: renamed from C2; value C_Polarized -> 150u
- C12: renamed from C3; value C_Polarized -> 150u
- R25: renamed from R1; value R -> 330
- U12: renamed from U11; symbol Interface_USB:CP2102N-Axx-xQFN20 -> Custom:CP2102N-Axx-xQFN20
- gave numbers to parts that had none: 22
- renumbered D2 to D1, D1 to D28, J2 to J1, J1 to J3, R2 to R1, R9 to R10, R3 to R2, R4 to R3, R8 to R9, U8 to U1, U1 to U10, U2 to U11, U4 to U2, U3 to U4, U6 to U7, U9 to U8, U7 to U9
Connections:
- net A0: now also J?.3 (Pin_3)
- net A1: now also J?.1 (Pin_1)
- net A11: now also U3.1 (A0)
- net A12: now also U3.2 (A1)
- net A13: now also U3.3 (A2)
- net A14: now also U3.5 (E2)
- net A15: now also U3.6 (E3); no longer U10.24 (CS1)
- net A2: now also J?.6 (Pin_6)
- net A3: now also J?.4 (Pin_4)
- net D0: now also J?.19 (Pin_19)
- net D1: now also J?.17 (Pin_17)
- net D2: now also J?.15 (Pin_15)
- net D3: now also J?.13 (Pin_13)
- net D4: now also J?.11 (Pin_11)
- net D5: now also J?.9 (Pin_9)
- net D6: now also J?.7 (Pin_7)
- net D7: now also J?.5 (Pin_5)
- net GND: now also C1.2, C11.2, C12.2, D28.1 (K), P1.A1 (GND), P1.A12 (GND), P1.B1 (GND), P1.B12 (GND), P1.S1 (SHIELD), U12.12 (GND), U12.21 (GND), U12.3 (GND), U2.7 (GND), U5.7 (GND), C10.2, C13.2, C14.2, C15.2, C16.2, C2.2, C3.2, C4.2, C5.2, C6.2, C7.2, C8.2, C9.2, D23.2 (A2), D24.2 (A2), D25.2 (A2), D26.2 (A2), D27.2 (A2), D29.2 (A2), D30.2 (A2), D31.2 (A2), D32.2 (A2), D33.1 (A1), D34.1 (A1), D35.1 (A1), J4.10 (Pin_10), J?.18 (Pin_18), J?.20 (Pin_20), R11.2, R12.2, R14.2, R27.2, R28.1, R4.2, U3.8 (GND)
- net NMIB: now also J2.1 (Pin_1)
- net PHI2: now also J?.10 (Pin_10)
- net RDB: now also J?.14 (Pin_14)
- net RESB: now also U2.11
- net RWB: now also J?.12 (Pin_12)
- net VDD: now also C1.1, C11.1, C12.1, P1.A4 (VBUS), P1.A9 (VBUS), P1.B4 (VBUS), P1.B9 (VBUS), R25.1, U12.7 (VREGIN), U2.14 (VCC), U5.14 (VCC), C10.1, C14.1, C16.1, C2.1, C3.1, C4.1, C5.1, C6.1, C7.1, C8.1, C9.1, D35.2 (A2), J?.2 (Pin_2), R13.1, R15.1, R16.1, R17.1, R18.1, R19.1, R20.1, R21.1, R22.1, R23.1, R24.1, R26.1, U3.16 (VCC)
- net WRB: now also J?.16 (Pin_16)
- net UARTCSB: now reaches U11.18 (~{CS})
- net UARTCSB: now also U3.14 (O1)
- net at U11.19 (~{MFB}): now also D27.1 (A1), J4.9 (Pin_9)
- net RES: now reaches U11.21 (RESET)
- net RES: now also U2.13
- net at U11.23 (~{RTSB}): now also D30.1 (A1), J4.6 (Pin_6)
- net at U11.25 (RXB): now also D31.1 (A1), J4.4 (Pin_4)
- net at U11.26 (TXB): now also D32.1 (A1), J4.2 (Pin_2)
- net at U11.27 (~{DTRB}): now also D26.1 (A1), J4.7 (Pin_7)
- net at U11.28 (~{CTSB}): now also D24.1 (A1), J4.3 (Pin_3), R19.2
- net at U11.29 (~{DSRB}): now also D25.1 (A1), J4.5 (Pin_5), R20.2
- net at U11.30 (~{CDB}): now also D23.1 (A1), J4.1 (Pin_1), R16.2
- net at U11.31 (~{RIB}): now also D29.1 (A1), J4.8 (Pin_8)
- net at U11.36 (~{RTSA}): now also U12.15 (~{CTS})
- net at U11.38 (TXA): now also U12.17 (RXD)
- net at U11.39 (RXA): now also U12.18 (TXD)
- net at U11.40 (~{CTSA}): now also U12.16 (~{RTS})
- net at U11.41 (~{DSRA}): now also U12.14 (SUSPEND), R22.2
- net at U11.42 (~{CDA}): now also R15.2
- net at U11.43 (~{RIA}): now also R17.2
- net at D28.2 (A): now also R25.2
- net at U5.10: now also R12.1
- net at U5.9: now also R11.1
- net at P1.A5 (CC): now also R28.2
- net at P1.A6 (D+): now also U12.4 (D+), D34.2 (A2)
- net at P1.A7 (D-): now also U12.5 (D-), D33.2 (A2)
- net at U10.21 (IRQB): now also J2.2 (Pin_2)
- net VIACSB: now reaches U10.23 (CS2B)
- net VIACSB: now also U3.15 (O0)
- net at U2.12: now also R14.1
- net at U12.13 (~{WAKEUP}): now also R23.2
- net at U12.19 (~{RXT}/GPIO.3): now also D22.1 (K)
- net at U12.20 (~{TXT}/GPIO.2): now also D21.1 (K)
- net 3V3: now reaches U12.6 (VDD)
- net 3V3: now also C13.1, C15.1
- net at U12.8 (VBUS): now also R26.2, R27.1
- net at U12.9 (~{RST}): now also R24.2
- net CA1 renamed IO.CA1
- net CA2 renamed IO.CA2
- net CB1 renamed IO.CB1
- net CB2 renamed IO.CB2
- net PA0 renamed IO.PA0
- net PA1 renamed IO.PA1
- net PA2 renamed IO.PA2
- net PA3 renamed IO.PA3
- net PA4 renamed IO.PA4
- net PA5 renamed IO.PA5
- net PA6 renamed IO.PA6
- net PA7 renamed IO.PA7
- net PB0 renamed IO.PB0
- net PB1 renamed IO.PB1
- net PB2 renamed IO.PB2
- net PB3 renamed IO.PB3
- net PB4 renamed IO.PB4
- net PB5 renamed IO.PB5
- net PB6 renamed IO.PB6
- net PB7 renamed IO.PB7
- new net: D21.2 (A), R18.2
- new net: R4.1, U3.4 (E1)
- new net: R13.2, U10.24 (CS1)
- new net: D22.2 (A), R21.2
- new net AUXCSB: J?.8 (Pin_8), U3.13 (O2)
- no-connect marks 8 -> 22
Other:
- note removed: "TODO"
- moved on the sheet: C1, C11, C12, D1, D10, D11, D12, D13, D14, D15, D16, D17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

Commit message: Assign footprints
Parts:
- D1, D10, D11, D12, D13, D14, D15, D16, D17, D18, D19, D2, D20, D23, D24, D25, D26, D27, D29, D3, D30, D31, D32, D33, D34, D35, D4, D5, D6, D7, D8, D9: footprint (none) -> Diode_SMD:D_0603_1608Metric_Pad1.05x0.95mm_HandSolder
- J1: renamed from J?; footprint (none) -> Connector_PinHeader_2.54mm:PinHeader_2x10_P2.54mm_Vertical
- J2: renamed from J1; footprint (none) -> Connector_PinHeader_2.54mm:PinHeader_1x03_P2.54mm_Vertical
- J3: renamed from J2; footprint (none) -> Connector_PinHeader_2.54mm:PinHeader_1x02_P2.54mm_Vertical
- J4: renamed from J3; footprint (none) -> Connector_PinHeader_2.54mm:PinHeader_2x20_P2.54mm_Vertical
- J5: renamed from J4; footprint (none) -> Connector_PinHeader_2.54mm:PinHeader_2x05_P2.54mm_Vertical
- U2: renamed from U3; footprint (none) -> Package_DIP:DIP-16_W7.62mm
- U4: renamed from U6; footprint Package_DIP:DIP-14_W7.62mm_Socket -> Package_DIP:DIP-14_W7.62mm
- U5: footprint Package_DIP:DIP-14_W7.62mm_Socket -> Package_DIP:DIP-14_W7.62mm
- renumbered U4 to U3, U7 to U6, U2 to U7

Commit message: Component placement and TVS routing finished
Parts:
- removed R10: 1k, Resistor_THT:R_Axial_DIN0207_L6.3mm_D2.5mm_P7.62mm_Horizontal, symbol Device:R
- added D36, D37, D38, D39, D40, D41, D42, D43, D44, D45, D46, D47, D48, D49, D50, D51, D52: D_TVS, Diode_SMD:D_0603_1608Metric_Pad1.05x0.95mm_HandSolder, symbol Device:D_TVS
- added H1, H2, H3, H4: MountingHole_Pad, MountingHole:MountingHole_4.3mm_M4_DIN965_Pad, symbol Mechanical:MountingHole_Pad
- C13, C14, C15, C16: footprint Capacitor_THT:C_Disc_D4.3mm_W1.9mm_P5.00mm -> Capacitor_SMD:C_0603_1608Metric_Pad1.08x0.95mm_HandSolder
Connections:
- net A0: now also D44.2 (A2)
- net A1: now also D45.2 (A2)
- net A2: now also D51.2 (A2)
- net A3: now also D52.2 (A2)
- net AUXCSB: now also D50.2 (A2)
- net D0: now also D36.2 (A2)
- net D1: now also D37.2 (A2)
- net D2: now also D38.2 (A2)
- net D3: now also D39.2 (A2)
- net D4: now also D40.2 (A2)
- net D5: now also D41.2 (A2)
- net D6: now also D42.2 (A2)
- net D7: now also D43.2 (A2)
- net GND: now also U9.1 (OE), D36.1 (A1), D37.1 (A1), D38.1 (A1), D39.1 (A1), D40.1 (A1), D41.1 (A1), D42.1 (A1), D43.1 (A1), D44.1 (A1), D45.1 (A1), D46.1 (A1), D47.1 (A1), D48.1 (A1), D49.1 (A1), D50.1 (A1), D51.1 (A1), D52.1 (A1), H1.1, H2.1, H3.1, H4.1
- net PHI2: now also D49.2 (A2)
- net RDB: now also D47.2 (A2)
- net RWB: now also D48.2 (A2)
- net WRB: now also D46.2 (A2)

Commit message: Remove extra 7400
Parts:
- removed R11, R12: 1k, Resistor_THT:R_Axial_DIN0207_L6.3mm_D2.5mm_P7.62mm_Horizontal, symbol Device:R
- removed U4: 74HC00, Package_DIP:DIP-14_W7.62mm, symbol 74xx:74HC00
- renumbered D36 to D1, D45 to D10, D46 to D11, D47 to D12, D48 to D13, D49 to D14, D50 to D15, D51 to D16, D52 to D17, D1 to D18, D2 to D19, D37 to D2, D3 to D20, D4 to D21, D5 to D22, D6 to D23, D7 to D24, D8 to D25, D9 to D26, D10 to D27, D11 to D28, D12 to D29, D38 to D3, D13 to D30, D14 to D31, D15 to D32, D16 to D33, D17 to D34, D18 to D35, D19 to D36, D20 to D37, D21 to D38, D22 to D39, D39 to D4, D23 to D40, D24 to D41, D25 to D42, D26 to D43, D27 to D44, D28 to D45, D29 to D46, D30 to D47, D31 to D48, D32 to D49, D40 to D5, D33 to D50, D34 to D51, D35 to D52, D41 to D6, D42 to D7, D43 to D8, D44 to D9, R13 to R10, R14 to R11, R15 to R12, R16 to R13, R17 to R14, R18 to R15, R19 to R16, R20 to R17, R21 to R18, R22 to R19, R23 to R20, R24 to R21, R25 to R22, R26 to R23, R27 to R24, R28 to R25, U11 to U10, U12 to U11, U5 to U4, U6 to U5, U7 to U6, U8 to U7, U9 to U8, U10 to U9
Connections:
- net D0: now also D8.2 (A2), J1.5 (Pin_5), U7.13 (DQ0); no longer D1.2 (A2), J1.19 (Pin_19), U7.21 (DQ7)
- net D1: now also D7.2 (A2), J1.7 (Pin_7), U7.14 (DQ1); no longer D2.2 (A2), J1.17 (Pin_17), U7.20 (DQ6)
- net D2: now also D6.2 (A2), J1.9 (Pin_9), U7.15 (DQ2); no longer D3.2 (A2), J1.15 (Pin_15), U7.19 (DQ5)
- net D3: now also D5.2 (A2), J1.11 (Pin_11), U7.17 (DQ3); no longer D4.2 (A2), J1.13 (Pin_13), U7.18 (DQ4)
- net D4: now also D4.2 (A2), J1.13 (Pin_13), U7.18 (DQ4); no longer D5.2 (A2), J1.11 (Pin_11), U7.17 (DQ3)
- net D5: now also D3.2 (A2), J1.15 (Pin_15), U7.19 (DQ5); no longer D6.2 (A2), J1.9 (Pin_9), U7.15 (DQ2)
- net D6: now also D2.2 (A2), J1.17 (Pin_17), U7.20 (DQ6); no longer D7.2 (A2), J1.7 (Pin_7), U7.14 (DQ1)
- net D7: now also D1.2 (A2), J1.19 (Pin_19), U7.21 (DQ7); no longer D8.2 (A2), J1.5 (Pin_5), U7.13 (DQ0)
- net PHI2: now also U4.10
- net RBW: now also U4.9
- net ~{WE}: now also U4.8
Other:
- moved on the sheet: U4C

Commit message: Complete initial routing
Parts:
- removed J1: Conn_02x10_Odd_Even, Connector_PinHeader_2.54mm:PinHeader_2x10_P2.54mm_Vertical, symbol Connector_Generic:Conn_02x10_Odd_Even
- added D18, D19, D20, D21: D_TVS, Diode_SMD:D_0603_1608Metric_Pad1.05x0.95mm_HandSolder, symbol Device:D_TVS
- added H1, H2: MountingHole_Pad, MountingHole:MountingHole_3.2mm_M3_Pad, symbol Mechanical:MountingHole_Pad
- added J1: Conn_02x12_Odd_Even, Connector_PinSocket_2.54mm:PinSocket_2x12_P2.54mm_Vertical, symbol Connector_Generic:Conn_02x12_Odd_Even
- H3: renamed from H1; footprint MountingHole:MountingHole_4.3mm_M4_DIN965_Pad -> MountingHole:MountingHole_3.2mm_M3_Pad
- H4: renamed from H2; footprint MountingHole:MountingHole_4.3mm_M4_DIN965_Pad -> MountingHole:MountingHole_3.2mm_M3_Pad
- H5: renamed from H3; footprint MountingHole:MountingHole_4.3mm_M4_DIN965_Pad -> MountingHole:MountingHole_3.2mm_M3_Pad
- H6: renamed from H4; footprint MountingHole:MountingHole_4.3mm_M4_DIN965_Pad -> MountingHole:MountingHole_3.2mm_M3_Pad
- renumbered D18 to D22, D19 to D23, D20 to D24, D21 to D25, D22 to D26, D23 to D27, D24 to D28, D25 to D29, D26 to D30, D27 to D31, D28 to D32, D29 to D33, D30 to D34, D31 to D35, D32 to D36, D33 to D37, D34 to D38, D35 to D39, D36 to D40, D37 to D41, D38 to D42, D39 to D43, D40 to D44, D41 to D45, D42 to D46, D43 to D47, D44 to D48, D45 to D49, D46 to D50, D47 to D51, D48 to D52, D49 to D53, D50 to D54, D51 to D55, D52 to D56, R4 to R2, R2 to R3, R3 to R4
Connections:
- net A0: now also U7.12 (A0), J1.6 (Pin_6); no longer U7.3 (A14)
- net A1: now also U7.11 (A1), J1.4 (Pin_4); no longer U7.28 (A13)
- net A10: now also U7.23 (A10); no longer U7.8 (A4)
- net A11: now also U7.25 (A11); no longer U7.9 (A3)
- net A12: now also U7.4 (A12); no longer U7.10 (A2)
- net A13: now also U7.28 (A13); no longer U7.11 (A1)
- net A14: now also U7.3 (A14); no longer U7.12 (A0)
- net A2: now also U7.10 (A2), D19.2 (A2), J1.5 (Pin_5); no longer D16.2 (A2), U7.4 (A12)
- net A3: now also U7.9 (A3), D20.2 (A2), J1.3 (Pin_3); no longer D17.2 (A2), U7.25 (A11)
- net A4: now also U7.8 (A4); no longer U7.23 (A10)
- net A5: now also U7.7 (A5); no longer U7.26 (A9)
- net A6: now also U7.6 (A6); no longer U7.27 (A8)
- net A8: now also U7.27 (A8); no longer U7.6 (A6)
- net A9: now also U7.26 (A9); no longer U7.7 (A5)
- net B0: now also U7.2 (A16); no longer U7.1 (A18)
- net B1: now also U7.1 (A18); no longer U7.30 (A17)
- net B2: now also U7.31 (A15); no longer U7.2 (A16)
- net B3: now also U7.30 (A17); no longer U7.31 (A15)
- net D0: now also J1.8 (Pin_8)
- net D1: now also J1.10 (Pin_10)
- net D2: now also J1.12 (Pin_12)
- net D3: now also J1.14 (Pin_14)
- net D4: now also J1.16 (Pin_16)
- net D5: now also J1.18 (Pin_18)
- net D6: now also J1.20 (Pin_20)
- net D7: now also J1.22 (Pin_22)
- net GND: now also D18.1 (A1), D19.1 (A1), D20.1 (A1), D21.1 (A1), H1.1, H2.1, J1.23 (Pin_23), J1.24 (Pin_24)
- net PHI2: now also D17.2 (A2), J1.15 (Pin_15); no longer D14.2 (A2)
- net RDB: now also J1.19 (Pin_19)
- net RWB: now also D18.2 (A2), J1.17 (Pin_17); no longer D13.2 (A2)
- net VDD: now also D21.2 (A2), J1.1 (Pin_1), J1.2 (Pin_2)
- net WRB: now also J1.21 (Pin_21)
- net AUXCSB1: now reaches U2.10 (O5)
- net AUXCSB1: now also D14.2 (A2), J1.9 (Pin_9)
- net AUXCSB0: now reaches U2.11 (O4)
- net AUXCSB0: now also D13.2 (A2), J1.7 (Pin_7)
- net AUXCSB3: now reaches U2.7 (O7)
- net AUXCSB3: now also D16.2 (A2), J1.13 (Pin_13)
- net AUXCSB2: now reaches U2.9 (O6)
- net AUXCSB2: now also D15.2 (A2), J1.11 (Pin_11)
- net AUXCSB: no longer names the net of U2.13 (O2)
- net AUXCSB: no longer D15.2 (A2)
- no-connect marks 22 -> 19
Other:
- note added: "/RDB"
- note added: "/RWB"
- note added: "/WRB"
- note added: "PHI2"
- moved on the sheet: C1, C10, C2, C3, C4, C5, C6, C7, C8, C9, D1, D10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
