File: minputer/minputer.kicad_sch (KiCad schematic)
At the start: 122 parts, among them J1 Conn_02x12_Odd_Even, J2 Conn_01x03_Male, J3 Conn_01x02_Male, J4 Conn_02x20_Odd_Even, J5 Conn_02x05_Odd_Even, P1 USB_C_Plug_USB2.0, SW1 SW_Push, U1 DS1318, U10 16C2552_PLCC, U11 CP2102N-Axx-xQFN20, U2 74LS138, U3 W65C816, U4 74HC00, U5 28C256, U6 74HC02, U7 AS6C4008-55PCN, U8 74LS573, U9 W65C22, X1 CXO_DIP8

Commit message: Add aux power input; reroute CP2102; add PHI2 osc
Parts:
- removed J3: Conn_01x02_Male, Connector_PinHeader_2.54mm:PinHeader_1x02_P2.54mm_Vertical, symbol Connector:Conn_01x02_Male
- added C17: 150u, Capacitor_THT:C_Radial_D8.0mm_H7.0mm_P3.50mm, symbol Device:C_Polarized
- added C18: 0.1u, Capacitor_SMD:C_0603_1608Metric_Pad1.08x0.95mm_HandSolder, symbol Device:C
- added D57: 1N4148, Diode_THT:D_DO-35_SOD27_P7.62mm_Horizontal, symbol Diode:1N4148
- added J3, J6: Conn_01x03_Male, Connector_PinHeader_2.54mm:PinHeader_1x03_P2.54mm_Vertical, symbol Connector:Conn_01x03_Male
- added J7: Barrel_Jack, Connector_BarrelJack:BarrelJack_Horizontal, symbol Connector:Barrel_Jack
- added J8: Screw_Terminal_01x02, TerminalBlock:TerminalBlock_bornier-2_P5.08mm, symbol Connector:Screw_Terminal_01x02
- added Q1: Q_PMOS_GDS, Package_TO_SOT_SMD:TO-263-3_TabPin2, symbol Device:Q_PMOS_GDS
- added U12: L7805, Package_TO_SOT_SMD:TO-263-3_TabPin2, symbol Regulator_Linear:L7805
- added X2: CXO_DIP8, Oscillator:Oscillator_DIP-8, symbol Oscillator:CXO_DIP8
- R19, R20, R21: footprint Resistor_THT:R_Axial_DIN0207_L6.3mm_D2.5mm_P7.62mm_Horizontal -> Resistor_SMD:R_0603_1608Metric_Pad0.98x0.95mm_HandSolder
Connections:
- net GND: now also C17.2, C18.2, J7.2, J8.2 (Pin_2), Q1.1 (G), U12.2 (GND), X2.4 (GND)
- net NMIB: now also J3.2 (Pin_2)
- net PHI2: now also X2.5 (OUT); no longer U10.13 (XTAL2)
- net VDD: now also J6.2 (Pin_2), X2.8 (Vcc); no longer C14.1, C16.1, D56.2 (A2), P1.A4 (VBUS), P1.A9 (VBUS), P1.B4 (VBUS), P1.B9 (VBUS), U11.7 (VREGIN)
- net at U9.21 (IRQB): now also J3.1 (Pin_1)
- new net: C18.1, D57.2 (A), J6.1 (Pin_1), U12.3 (OUT)
- new net: C14.1, C16.1, D56.2 (A2), J6.3 (Pin_3), P1.A4 (VBUS), P1.A9 (VBUS), P1.B4 (VBUS), P1.B9 (VBUS), U11.7 (VREGIN)
- new net: C17.1, D57.1 (K), Q1.3 (S), U12.1 (IN)
- new net PWR_IN: J7.1, J8.1 (Pin_1), Q1.2 (D)
- no-connect marks 19 -> 21
Other:
- note added: "Alternate Power Input Regulator"
- note added: "Alternative Power Inputs Recommended: +7V to +15V Abs. Max: -30V to +30V"
- note added: "Power Selection (USB or Alternate)"
- note added: "Reverse Polarity Protection"
- moved on the sheet: R1, SW1, U1

Commit message: Add GND TPs; generate logo symbol/model files
Parts:
- added D19: D_TVS, Diode_SMD:D_0603_1608Metric_Pad1.05x0.95mm_HandSolder, symbol Device:D_TVS
- added G1: LOGO, symbol zediac-logo:LOGO
- added TP1, TP2: TestPoint, TestPoint:TestPoint_Bridge_Pitch2.54mm_Drill1.0mm, symbol Connector:TestPoint
- renumbered C12 to C1, C6 to C10, C10 to C12, C18 to C13, C17 to C14, C13 to C15, C15 to C17, C14 to C18, C8 to C2, C9 to C3, C1 to C4, C2 to C5, C4 to C6, C3 to C7, C7 to C8, C5 to C9, D43 to D1, D46 to D10, D45 to D11, D44 to D12, D51 to D13, D53 to D14, D52 to D15, D50 to D16, D15 to D17, D19 to D18, D57 to D2, D10 to D20, D20 to D21, D9 to D22, D21 to D23, D14 to D24, D13 to D25, D8 to D26, D16 to D27, D7 to D28, D5 to D29, D56 to D3, D17 to D30, D12 to D31, D11 to D32, D6 to D33, D4 to D34, D2 to D35, D1 to D36, D18 to D37, D3 to D38, D23 to D39, D49 to D4, D29 to D40, D22 to D41, D27 to D42, D25 to D43, D30 to D44, D28 to D45, D24 to D46, D31 to D47, D26 to D48, D36 to D49, D54 to D5, D33 to D50, D38 to D51, D35 to D52, D41 to D53, D37 to D54, D40 to D55, D39 to D56, D32 to D57, D34 to D58, D42 to D6, D55 to D7, D48 to D8, D47 to D9, H6 to H1, H5 to H2, H1 to H3, H2 to H4, H3 to H5, H4 to H6, J4 to J1, J3 to J2, J1 to J3, J2 to J4, J8 to J7, J7 to J8, R3 to R1, R9 to R10, R18 to R11, R7 to R12, R17 to R13, R16 to R14, R14 to R15, R12 to R16, R2 to R17, R13 to R18, R21 to R19, R4 to R2, R19 to R20, R22 to R21, R25 to R22, R24 to R23, R20 to R24, R23 to R25, R5 to R3, R6 to R4, R1 to R5, R15 to R6, R10 to R7, R11 to R9, U9 to U1, U2 to U10, U12 to U11, U11 to U12, U1 to U2, U7 to U4, U8 to U7, U10 to U8, U4 to U9
Connections:
- net GND: now also D19.1 (A1), TP1.1, TP2.1
- net VDD: no longer J3.2 (Pin_2)
- net /RDY: now reaches R3.2, U3.2 (RDY)
- net /RDY: now also J3.2 (Pin_2), D19.2 (A2)
Other:
- moved on the sheet: D20, D22, D26, D28, D29, D33, D34, D35, D36, D38
