File: zediac/zediac.kicad_sch (KiCad schematic)
At the start: 138 parts, among them J1 Conn_02x20_Odd_Even, J2 Conn_01x03_Male, J3 Conn_02x12_Odd_Even, J4 Conn_01x03_Male, J5 Conn_02x05_Odd_Even, J6 Conn_01x03_Male, J7 Screw_Terminal_01x02, J8 Barrel_Jack, P1 USB_C_Plug_USB2.0, Q1 Q_PMOS_GDS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

Commit message: [pcb] Add reset jumper/header
Parts:
- added J9: Conn_01x02_Pin, Connector_PinHeader_2.54mm:PinHeader_1x02_P2.54mm_Vertical, symbol Connector:Conn_01x02_Pin
Connections:
- net GND: now also J9.2 (Pin_2)
- net RESB: now also J9.1 (Pin_1)
Changed lines of the file:
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@@
   (junction (at 347.98 275.59) (diameter 0) (color 0 0 0 0)
   )
+  (junction (at 20.955 149.86) (diameter 0) (color 0 0 0 0)
+  )
   (junction (at 100.33 309.88) (diameter 0) (color 0 0 0 0)
   )
@@
   (junction (at 127 161.29) (diameter 0) (color 0 0 0 0)
   )
+  (junction (at 37.465 137.16) (diameter 0) (color 0 0 0 0)
+  )
   (junction (at 39.37 309.88) (diameter 0) (color 0 0 0 0)
   )
@@
     (stroke (width 0) (type default))
   )
+  (wire (pts (xy 20.955 149.86) (xy 20.955 154.94))
+    (stroke (width 0) (type default))
+  )
   (wire (pts (xy 187.96 213.36) (xy 396.24 213.36))
     (stroke (width 0) (type default))
@@
     (stroke (width 0) (type default))
   )
+  (wire (pts (xy 29.845 147.955) (xy 29.845 149.86))
+    (stroke (width 0) (type default))
+  )
   (wire (pts (xy 289.56 156.21) (xy 306.07 156.21))
     (stroke (width 0) (type default))
@@
     (stroke (width 0) (type default))
   )
+  (wire (pts (xy 27.305 149.86) (xy 20.955 149.86))
+    (stroke (width 0) (type default))
+  )
   (wire (pts (xy 537.21 53.34) (xy 537.21 62.23))
     (stroke (width 0) (type default))
@@
     (stroke (width 0) (type default))
   )
-  (wire (pts (xy 20.955 137.16) (xy 20.955 139.7))
+  (wire (pts (xy 20.955 137.16) (xy 20.955 149.86))
     (stroke (width 0) (type default))
   )
@@
     (stroke (width 0) (type default))
   )
+  (wire (pts (xy 29.845 149.86) (xy 37.465 149.86))
+    (stroke (width 0) (type default))
+  )
   (bus (pts (xy 283.21 142.24) (xy 283.21 144.78))
     (stroke (width 0) (type default))
@@
     (stroke (width 0) (type default))
   )
+  (wire (pts (xy 27.305 147.955) (xy 27.305 149.86))
+    (stroke (width 0) (type default))
+  )
   (bus (pts (xy 199.39 255.27) (xy 199.39 252.73))
     (stroke (width 0) (type default))
@@
     (stroke (width 0) (type default))
   )
+  (wire (pts (xy 37.465 149.86) (xy 37.465 137.16))
+    (stroke (width 0) (type default))
+  )
   (bus (pts (xy 199.39 260.35) (xy 199.39 257.81))
     (stroke (width 0) (type default))
@@
     )
   )
-  (symbol (lib_id "power:GND") (at 20.955 139.7 0) (unit 1)
+  (symbol (lib_id "power:GND") (at 20.955 154.94 0) (unit 1)
     (in_bom yes) (on_board yes) (dnp no) (fields_autoplaced)
-    (property "Reference" "#PWR02" (at 20.955 146.05 0)
+    (property "Reference" "#PWR02" (at 20.955 161.29 0)
       (effects (font (size 1.27 1.27)) hide)
     )
-    (property "Value" "GND" (at 20.955 146.05 0)
+    (property "Value" "GND" (at 20.955 161.29 0)
       (effects (font (size 1.27 1.27)))
     )
-    (property "Footprint" "" (at 20.955 139.7 0)
+    (property "Footprint" "" (at 20.955 154.94 0)
       (effects (font (size 1.27 1.27)) hide)
     )
-    (property "Datasheet" "" (at 20.955 139.7 0)
+    (property "Datasheet" "" (at 20.955 154.94 0)
       (effects (font (size 1.27 1.27)) hide)
     )
@@
         )
       )
+    )
+  )
+  (symbol (lib_id "Connector:Conn_01x02_Pin") (at 29.845 142.875 270) (unit 1)
+    (in_bom yes) (on_board yes) (dnp no)
+    (property "Reference" "J9" (at 26.67 154.305 90)
+      (effects (font (size 1.27 1.27)) (justify left))
+    )
+    (property "Value" "Conn_01x02_Pin" (at 22.225 151.765 90)
+      (effects (font (size 1.27 1.27)) (justify left))
+    )
+    (property "Footprint" "Connector_PinHeader_2.54mm:PinHeader_1x02_P2.54mm_Vertical" (at 29.845 142.875 0)
+      (effects (font (size 1.27 1.27)) hide)
+    )
+    (property "Datasheet" "~" (at 29.845 142.875 0)
+      (effects (font (size 1.27 1.27)) hide)
+    )
+    (pin "1")
+    (pin "2")
+    (instances
+      (project "zediac"
+        (path "/66a26b62-9544-494f-a4ed-13e8e346800a"
+          (reference "J9") (unit 1)
+        )
+      )

Commit message: [pcb] Add TVS to reset line
Parts:
- added D59: D_TVS, Diode_SMD:D_0603_1608Metric_Pad1.05x0.95mm_HandSolder, symbol Device:D_TVS
Connections:
- net GND: now also D59.1 (A1)
- net RESB: now also D59.2 (A2)
Changed lines of the file:
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@@
   (junction (at 367.03 318.77) (diameter 0) (color 0 0 0 0)
   )
+  (junction (at 37.465 149.86) (diameter 0) (color 0 0 0 0)
+  )
   (junction (at 33.655 352.425) (diameter 0) (color 0 0 0 0)
   )
@@
   (junction (at 512.445 43.815) (diameter 0) (color 0 0 0 0)
   )
+  (junction (at 20.955 158.115) (diameter 0) (color 0 0 0 0)
+  )
   (junction (at 506.73 107.95) (diameter 0) (color 0 0 0 0)
   )
@@
     (stroke (width 0) (type default))
   )
+  (wire (pts (xy 37.465 158.115) (xy 37.465 149.86))
+    (stroke (width 0) (type default))
+  )
   (wire (pts (xy 72.39 314.96) (xy 82.55 314.96))
     (stroke (width 0) (type default))
@@
     (stroke (width 0) (type default))
   )
-  (wire (pts (xy 20.955 149.86) (xy 20.955 154.94))
+  (wire (pts (xy 20.955 149.86) (xy 20.955 158.115))
     (stroke (width 0) (type default))
   )
@@
     (stroke (width 0) (type default))
   )
+  (wire (pts (xy 20.955 158.115) (xy 20.955 161.29))
+    (stroke (width 0) (type default))
+  )
   (wire (pts (xy 519.43 147.32) (xy 519.43 100.33))
     (stroke (width 0) (type default))
@@
     (stroke (width 0) (type default))
   )
+  (wire (pts (xy 32.385 158.115) (xy 37.465 158.115))
+    (stroke (width 0) (type default))
+  )
   (wire (pts (xy 20.955 115.57) (xy 20.955 119.38))
     (stroke (width 0) (type default))
@@
     (stroke (width 0) (type default))
   )
+  (wire (pts (xy 20.955 158.115) (xy 24.765 158.115))
+    (stroke (width 0) (type default))
+  )
   (wire (pts (xy 377.825 160.02) (xy 377.825 165.735))
     (stroke (width 0) (type default))
@@
     )
   )
+  (symbol (lib_id "Device:D_TVS") (at 28.575 158.115 0) (unit 1)
+    (in_bom yes) (on_board yes) (dnp no)
+    (property "Reference" "D59" (at 30.48 160.655 0)
+      (effects (font (size 1.27 1.27)) (justify right))
+    )
+    (property "Value" "D_TVS" (at 27.3051 160.655 90)
+      (effects (font (size 1.27 1.27)) (justify right) hide)
+    )
+    (property "Footprint" "Diode_SMD:D_0603_1608Metric_Pad1.05x0.95mm_HandSolder" (at 28.575 158.115 0)
+      (effects (font (size 1.27 1.27)) hide)
+    )
+    (property "Datasheet" "~" (at 28.575 158.115 0)
+      (effects (font (size 1.27 1.27)) hide)
+    )
+    (pin "1")
+    (pin "2")
+    (instances
+      (project "zediac"
+        (path "/66a26b62-9544-494f-a4ed-13e8e346800a"
+          (reference "D59") (unit 1)
+        )
+      )
+    )
+  )
   (symbol (lib_id "power:GND") (at 148.59 339.09 0) (unit 1)
     (in_bom yes) (on_board yes) (dnp no)
@@
     )
   )
-  (symbol (lib_id "power:GND") (at 20.955 154.94 0) (unit 1)
+  (symbol (lib_id "power:GND") (at 20.955 161.29 0) (unit 1)
     (in_bom yes) (on_board yes) (dnp no) (fields_autoplaced)
-    (property "Reference" "#PWR02" (at 20.955 161.29 0)
+    (property "Reference" "#PWR02" (at 20.955 167.64 0)
       (effects (font (size 1.27 1.27)) hide)
     )
-    (property "Value" "GND" (at 20.955 161.29 0)
+    (property "Value" "GND" (at 20.955 167.64 0)
       (effects (font (size 1.27 1.27)))
     )
-    (property "Footprint" "" (at 20.955 154.94 0)
+    (property "Footprint" "" (at 20.955 161.29 0)
       (effects (font (size 1.27 1.27)) hide)
     )
-    (property "Datasheet" "" (at 20.955 154.94 0)
+    (property "Datasheet" "" (at 20.955 161.29 0)
       (effects (font (size 1.27 1.27)) hide)
     )
