File: expansion-boards/template/zediac-template.kicad_pcb (KiCad board)
At the start: 4 copper layers, 150 x 90 mm, 12 parts, among them J3 Conn_02x12_Odd_Even

Commit message: [exp-template] Correct template; Create template rename script
Parts:
- G1: footprint zediac:zediac-logo -> zediac-template:zediac-template-logo
Changed lines of the file:
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@@
 		(property ki_fp_filters "LED* LED_SMD:* LED_THT:*")
 		(sheetname "Root")
-		(sheetfile "zediac-template.kicad_sch")
+		(sheetfile "zediac-template-template.kicad_sch")
 		(attr through_hole)
 		(fp_line
@@
 		(property ki_fp_filters "R_*")
 		(sheetname "Root")
-		(sheetfile "zediac-template.kicad_sch")
+		(sheetfile "zediac-template-template.kicad_sch")
 		(attr through_hole)
 		(fp_line
@@
 		(property ki_fp_filters "MountingHole*Pad*")
 		(sheetname "Root")
-		(sheetfile "zediac-template.kicad_sch")
+		(sheetfile "zediac-template-template.kicad_sch")
 		(attr exclude_from_pos_files)
 		(fp_circle
@@
 		(property ki_fp_filters "MountingHole*Pad*")
 		(sheetname "Root")
-		(sheetfile "zediac-template.kicad_sch")
+		(sheetfile "zediac-template-template.kicad_sch")
 		(attr exclude_from_pos_files)
 		(fp_circle
@@
 		(property ki_fp_filters "MountingHole*Pad*")
 		(sheetname "Root")
-		(sheetfile "zediac-template.kicad_sch")
+		(sheetfile "zediac-template-template.kicad_sch")
 		(attr exclude_from_pos_files)
 		(fp_circle
@@
 		(property ki_fp_filters "MountingHole*Pad*")
 		(sheetname "Root")
-		(sheetfile "zediac-template.kicad_sch")
+		(sheetfile "zediac-template-template.kicad_sch")
 		(attr exclude_from_pos_files)
 		(fp_circle
@@
 		(property ki_fp_filters "CP_*")
 		(sheetname "Root")
-		(sheetfile "zediac-template.kicad_sch")
+		(sheetfile "zediac-template-template.kicad_sch")
 		(attr through_hole)
 		(fp_circle
@@
 		(property ki_fp_filters "MountingHole*Pad*")
 		(sheetname "Root")
-		(sheetfile "zediac-template.kicad_sch")
+		(sheetfile "zediac-template-template.kicad_sch")
 		(attr exclude_from_pos_files)
 		(fp_circle
@@
 		(property ki_fp_filters "CP_*")
 		(sheetname "Root")
-		(sheetfile "zediac-template.kicad_sch")
+		(sheetfile "zediac-template-template.kicad_sch")
 		(attr through_hole)
 		(fp_circle
@@
 		)
 	)
-	(footprint "zediac:zediac-logo"
+	(footprint "zediac-template:zediac-template-logo"
 		(layer "F.Cu")
 		(at 149.86 106.68)
@@
 			)
 		)
-		(property "Footprint" "zediac:zediac-logo"
+		(property "Footprint" "zediac-template:zediac-template-logo"
 			(at 0 0 0)
 			(unlocked yes)
@@
 		)
 		(sheetname "Root")
-		(sheetfile "zediac-template.kicad_sch")
+		(sheetfile "zediac-template-template.kicad_sch")
 		(attr exclude_from_pos_files)
 		(fp_poly
@@
 		(property ki_fp_filters "Connector*:*_2x??_*")
 		(sheetname "Root")
-		(sheetfile "zediac-template.kicad_sch")
+		(sheetfile "zediac-template-template.kicad_sch")
 		(attr through_hole)
 		(fp_line
@@
 		(property ki_fp_filters "MountingHole*Pad*")
 		(sheetname "Root")
-		(sheetfile "zediac-template.kicad_sch")
+		(sheetfile "zediac-template-template.kicad_sch")
 		(attr exclude_from_pos_files)
 		(fp_circle

Commit message: [exp-template] Fix template sch/pcb connection errors
Parts:
- removed D4: LED, LED_THT:LED_D5.0mm
- removed R21: 330, Resistor_THT:R_Axial_DIN0207_L6.3mm_D2.5mm_P7.62mm_Horizontal
- G1: footprint zediac-template:zediac-template-logo -> zediac:zediac-logo
