File: expansion-boards/template/zediac-template.kicad_sch (KiCad schematic)
At the start: 10 parts, among them J3 Conn_02x12_Odd_Even

Commit message: [exp-template] Correct template; Create template rename script
Parts:
- G1: footprint zediac:zediac-logo -> zediac-template:zediac-template-logo; symbol zediac-logo:LOGO -> zediac-template-logo:LOGO
Changed lines of the file:
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@@
 		)
 		(instances
-			(project "zediac-template"
+			(project "zediac-template-template"
 				(path "/66a26b62-9544-494f-a4ed-13e8e346800a"
 					(reference "#PWR064")
@@
 		)
 		(instances
-			(project "zediac-template"
+			(project "zediac-template-template"
 				(path "/66a26b62-9544-494f-a4ed-13e8e346800a"
 					(reference "H3")
@@
 		)
 		(instances
-			(project "zediac-template"
+			(project "zediac-template-template"
 				(path "/66a26b62-9544-494f-a4ed-13e8e346800a"
 					(reference "H2")
@@
 		)
 		(instances
-			(project "zediac-template"
+			(project "zediac-template-template"
 				(path "/66a26b62-9544-494f-a4ed-13e8e346800a"
 					(reference "#PWR013")
@@
 		)
 		(instances
-			(project "zediac-template"
+			(project "zediac-template-template"
 				(path "/66a26b62-9544-494f-a4ed-13e8e346800a"
 					(reference "C11")
@@
 		)
 		(instances
-			(project "zediac-template"
+			(project "zediac-template-template"
 				(path "/66a26b62-9544-494f-a4ed-13e8e346800a"
 					(reference "#PWR068")
@@
 		)
 		(instances
-			(project "zediac-template"
+			(project "zediac-template-template"
 				(path "/66a26b62-9544-494f-a4ed-13e8e346800a"
 					(reference "#PWR073")
@@
 		)
 		(instances
-			(project "zediac-template"
+			(project "zediac-template-template"
 				(path "/66a26b62-9544-494f-a4ed-13e8e346800a"
 					(reference "#PWR065")
@@
 		)
 		(instances
-			(project "zediac-template"
+			(project "zediac-template-template"
 				(path "/66a26b62-9544-494f-a4ed-13e8e346800a"
 					(reference "#PWR074")
@@
 		)
 		(instances
-			(project "zediac-template"
+			(project "zediac-template-template"
 				(path "/66a26b62-9544-494f-a4ed-13e8e346800a"
 					(reference "#PWR067")
@@
 		)
 		(instances
-			(project "zediac-template"
+			(project "zediac-template-template"
 				(path "/66a26b62-9544-494f-a4ed-13e8e346800a"
 					(reference "H5")
@@
 		)
 		(instances
-			(project "zediac-template"
+			(project "zediac-template-template"
 				(path "/66a26b62-9544-494f-a4ed-13e8e346800a"
 					(reference "H4")
@@
 		)
 		(instances
-			(project "zediac-template"
+			(project "zediac-template-template"
 				(path "/66a26b62-9544-494f-a4ed-13e8e346800a"
 					(reference "#PWR080")
@@
 	)
 	(symbol
-		(lib_id "zediac-logo:LOGO")
+		(lib_id "zediac-template-logo:LOGO")
 		(at 494.03 360.68 0)
 		(unit 1)
@@
 			)
 		)
-		(property "Footprint" "zediac:zediac-logo"
+		(property "Footprint" "zediac-template:zediac-template-logo"
 			(at 494.03 360.68 0)
 			(effects
@@
 		)
 		(instances
-			(project "zediac-template"
+			(project "zediac-template-template"
 				(path "/66a26b62-9544-494f-a4ed-13e8e346800a"
 					(reference "G1")
@@
 		)
 		(instances
-			(project "zediac-template"
+			(project "zediac-template-template"
 				(path "/66a26b62-9544-494f-a4ed-13e8e346800a"
 					(reference "#PWR014")
@@
 		)
 		(instances
-			(project "zediac-template"
+			(project "zediac-template-template"
 				(path "/66a26b62-9544-494f-a4ed-13e8e346800a"
 					(reference "H1")
@@
 		)
 		(instances
-			(project "zediac-template"
+			(project "zediac-template-template"
 				(path "/66a26b62-9544-494f-a4ed-13e8e346800a"
 					(reference "H6")
@@
 		)
 		(instances
-			(project "zediac-template"
+			(project "zediac-template-template"
 				(path "/66a26b62-9544-494f-a4ed-13e8e346800a"
 					(reference "C1")
@@
 		)
 		(instances
-			(project "zediac-template"
+			(project "zediac-template-template"
 				(path "/66a26b62-9544-494f-a4ed-13e8e346800a"
 					(reference "#PWR079")
@@
 		)
 		(instances
-			(project "zediac-template"
+			(project "zediac-template-template"
 				(path "/66a26b62-9544-494f-a4ed-13e8e346800a"
 					(reference "J3")

Commit message: [exp-template] Fix template sch/pcb connection errors
Parts:
- G1: footprint zediac-template:zediac-template-logo -> zediac:zediac-logo; symbol zediac-template-logo:LOGO -> zediac-logo:LOGO
Changed lines of the file:
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@@
 		)
 		(instances
-			(project "zediac-template-template"
+			(project "zediac"
 				(path "/66a26b62-9544-494f-a4ed-13e8e346800a"
 					(reference "#PWR064")
@@
 		)
 		(instances
-			(project "zediac-template-template"
+			(project "zediac"
 				(path "/66a26b62-9544-494f-a4ed-13e8e346800a"
 					(reference "H3")
@@
 		)
 		(instances
-			(project "zediac-template-template"
+			(project "zediac"
 				(path "/66a26b62-9544-494f-a4ed-13e8e346800a"
 					(reference "H2")
@@
 		)
 		(instances
-			(project "zediac-template-template"
+			(project "zediac"
 				(path "/66a26b62-9544-494f-a4ed-13e8e346800a"
 					(reference "#PWR013")
@@
 		)
 		(instances
-			(project "zediac-template-template"
+			(project "zediac"
 				(path "/66a26b62-9544-494f-a4ed-13e8e346800a"
 					(reference "C11")
@@
 		)
 		(instances
-			(project "zediac-template-template"
+			(project "zediac"
 				(path "/66a26b62-9544-494f-a4ed-13e8e346800a"
 					(reference "#PWR068")
@@
 		)
 		(instances
-			(project "zediac-template-template"
+			(project "zediac"
 				(path "/66a26b62-9544-494f-a4ed-13e8e346800a"
 					(reference "#PWR073")
@@
 		)
 		(instances
-			(project "zediac-template-template"
+			(project "zediac"
 				(path "/66a26b62-9544-494f-a4ed-13e8e346800a"
 					(reference "#PWR065")
@@
 		)
 		(instances
-			(project "zediac-template-template"
+			(project "zediac"
 				(path "/66a26b62-9544-494f-a4ed-13e8e346800a"
 					(reference "#PWR074")
@@
 		)
 		(instances
-			(project "zediac-template-template"
+			(project "zediac"
 				(path "/66a26b62-9544-494f-a4ed-13e8e346800a"
 					(reference "#PWR067")
@@
 		)
 		(instances
-			(project "zediac-template-template"
+			(project "zediac"
 				(path "/66a26b62-9544-494f-a4ed-13e8e346800a"
 					(reference "H5")
@@
 		)
 		(instances
-			(project "zediac-template-template"
+			(project "zediac"
 				(path "/66a26b62-9544-494f-a4ed-13e8e346800a"
 					(reference "H4")
@@
 		)
 		(instances
-			(project "zediac-template-template"
+			(project "zediac"
 				(path "/66a26b62-9544-494f-a4ed-13e8e346800a"
 					(reference "#PWR080")
@@
 	)
 	(symbol
-		(lib_id "zediac-template-logo:LOGO")
+		(lib_id "zediac-logo:LOGO")
 		(at 494.03 360.68 0)
 		(unit 1)
@@
 			)
 		)
-		(property "Footprint" "zediac-template:zediac-template-logo"
+		(property "Footprint" "zediac:zediac-logo"
 			(at 494.03 360.68 0)
 			(effects
@@
 		)
 		(instances
-			(project "zediac-template-template"
+			(project "zediac"
 				(path "/66a26b62-9544-494f-a4ed-13e8e346800a"
 					(reference "G1")
@@
 		)
 		(instances
-			(project "zediac-template-template"
+			(project "zediac"
 				(path "/66a26b62-9544-494f-a4ed-13e8e346800a"
 					(reference "#PWR014")
@@
 		)
 		(instances
-			(project "zediac-template-template"
+			(project "zediac"
 				(path "/66a26b62-9544-494f-a4ed-13e8e346800a"
 					(reference "H1")
@@
 		)
 		(instances
-			(project "zediac-template-template"
+			(project "zediac"
 				(path "/66a26b62-9544-494f-a4ed-13e8e346800a"
 					(reference "H6")
@@
 		)
 		(instances
-			(project "zediac-template-template"
+			(project "zediac"
 				(path "/66a26b62-9544-494f-a4ed-13e8e346800a"
 					(reference "C1")
@@
 		)
 		(instances
-			(project "zediac-template-template"
+			(project "zediac"
 				(path "/66a26b62-9544-494f-a4ed-13e8e346800a"
 					(reference "#PWR079")
@@
 		)
 		(instances
-			(project "zediac-template-template"
+			(project "zediac"
 				(path "/66a26b62-9544-494f-a4ed-13e8e346800a"
 					(reference "J3")
